Commit message: Attach receptacle to world through a fixed joint and at a certain height above the ground.

File: planar_folding_assembly/urdf/receptacle.urdf.xacro (robot description, xacro)
@@ -6,4 +6,10 @@
   <xacro:property name="receptacle_h" value="0.05" />
   <xacro:property name="handle_distance" value="0.01" />
+  <link name="world" />
+  <joint name="base_receptacle_joint" type="fixed">
+    <origin xyz="0 0 0.2" />
+    <parent link="world" />
+    <child link="receptacle_handle" />
+  </joint>
   <link name="receptacle_handle" >
     <collision>
@@ -66,3 +72,7 @@
     </inertial>
   </link>
+  <gazebo>
+    <plugin name="test_receptacle_force" filename="libgazebo_ros_test_receptacle_force.so">
+    </plugin>
+  </gazebo>
 </robot>
